File: reed_fix/reed_fix.kicad_pcb (KiCad board)
At the start: 2 copper layers, 12.1 x 15.2 mm, 2 parts, among them J1 Conn_01x02_Male, SW1 SW_Reed

Commit message: spacer
Other:
- outline, holes or cut-outs redrawn
- board text added: "IN"
- board text removed: "OUT"
