File: port_expander/port_expander.kicad_pcb (KiCad board)
At the start: 2 copper layers, 110 x 110 mm, 33 parts, among them J0 Conn_02x08_Male, J1 Conn_02x08_Male, J10 Display, J11 Power, J12 SD, J13 Dial, J2 Conn_02x08_Male, J3 Conn_02x08_Male, J4 Conn_02x08_Male, J5 Conn_02x08_Male, J6 Conn_02x08_Male, J7 Conn_02x08_Male, J8 Conn_02x08_Male, J9 Conn_02x08_Male, Q1 BC548, U1 74HC32

Commit message: diode on buzzer
Parts:
- added D1: 1N4007, Diode_THT:D_DO-41_SOD81_P7.62mm_Horizontal, F.Cu at (112.4, 96.9)
Routing:
- net Net-(BZ1-Pad1): track 14.6 -> 30.3 mm
- net Net-(BZ1-Pad2): track 12.7 -> 28.3 mm
Changed lines of the file:
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@@
-(kicad_pcb (version 20171130) (host pcbnew "(5.1.8-0-10_14)")
+(kicad_pcb (version 20171130) (host pcbnew "(5.1.9)-1")
   (general
     (thickness 1.6)
     (drawings 119)
-    (tracks 853)
+    (tracks 857)
     (zones 0)
-    (modules 33)
+    (modules 34)
     (nets 146)
   )
@@
     (add_net GND)
   )
+  (module Diode_THT:D_DO-41_SOD81_P7.62mm_Horizontal (layer F.Cu)
+    (at 112.435 96.864 90)
+    (descr "Diode, DO-41_SOD81 series, Axial, Horizontal, pin pitch=7.62mm, , length*diameter=5.2*2.7mm^2, , http://www.diodes.com/_files/packages/DO-41%20(Plastic).pdf")
+    (tags "Diode DO-41_SOD81 series Axial Horizontal pin pitch 7.62mm  length 5.2mm diameter 2.7mm")
+    (fp_text reference D1 (at 3.81 -2.47 90) (layer F.SilkS)
+      (effects (font (size 1 1) (thickness 0.15)))
+    )
+    (fp_text value 1N4007 (at 3.81 2.47 90) (layer F.Fab)
+      (effects (font (size 1 1) (thickness 0.15)))
+    )
+    (fp_line (start 8.97 -1.6) (end -1.35 -1.6) (layer F.CrtYd) (width 0.05))
+    (fp_line (start 8.97 1.6) (end 8.97 -1.6) (layer F.CrtYd) (width 0.05))
+    (fp_line (start -1.35 1.6) (end 8.97 1.6) (layer F.CrtYd) (width 0.05))
+    (fp_line (start -1.35 -1.6) (end -1.35 1.6) (layer F.CrtYd) (width 0.05))
+    (fp_line (start 1.87 -1.47) (end 1.87 1.47) (layer F.SilkS) (width 0.12))
+    (fp_line (start 2.11 -1.47) (end 2.11 1.47) (layer F.SilkS) (width 0.12))
+    (fp_line (start 1.99 -1.47) (end 1.99 1.47) (layer F.SilkS) (width 0.12))
+    (fp_line (start 6.53 1.47) (end 6.53 1.34) (layer F.SilkS) (width 0.12))
+    (fp_line (start 1.09 1.47) (end 6.53 1.47) (layer F.SilkS) (width 0.12))
+    (fp_line (start 1.09 1.34) (end 1.09 1.47) (layer F.SilkS) (width 0.12))
+    (fp_line (start 6.53 -1.47) (end 6.53 -1.34) (layer F.SilkS) (width 0.12))
+    (fp_line (start 1.09 -1.47) (end 6.53 -1.47) (layer F.SilkS) (width 0.12))
+    (fp_line (start 1.09 -1.34) (end 1.09 -1.47) (layer F.SilkS) (width 0.12))
+    (fp_line (start 1.89 -1.35) (end 1.89 1.35) (layer F.Fab) (width 0.1))
+    (fp_line (start 2.09 -1.35) (end 2.09 1.35) (layer F.Fab) (width 0.1))
+    (fp_line (start 1.99 -1.35) (end 1.99 1.35) (layer F.Fab) (width 0.1))
+    (fp_line (start 7.62 0) (end 6.41 0) (layer F.Fab) (width 0.1))
+    (fp_line (start 0 0) (end 1.21 0) (layer F.Fab) (width 0.1))
+    (fp_line (start 6.41 -1.35) (end 1.21 -1.35) (layer F.Fab) (width 0.1))
+    (fp_line (start 6.41 1.35) (end 6.41 -1.35) (layer F.Fab) (width 0.1))
+    (fp_line (start 1.21 1.35) (end 6.41 1.35) (layer F.Fab) (width 0.1))
+    (fp_line (start 1.21 -1.35) (end 1.21 1.35) (layer F.Fab) (width 0.1))
+    (fp_text user K (at 0 -2.413 90) (layer F.SilkS)
+      (effects (font (size 1 1) (thickness 0.15)))
+    )
+    (fp_text user K (at 0 -2.1 90) (layer F.Fab)
+      (effects (font (size 1 1) (thickness 0.15)))
+    )
+    (fp_text user %R (at 4.2 0 90) (layer F.Fab)
+      (effects (font (size 1 1) (thickness 0.15)))
+    )
+    (pad 2 thru_hole oval (at 7.62 0 90) (size 2.2 2.2) (drill 1.1) (layers *.Cu *.Mask)
+      (net 130 "Net-(BZ1-Pad2)"))
+    (pad 1 thru_hole rect (at 0 0 90) (size 2.2 2.2) (drill 1.1) (layers *.Cu *.Mask)
+      (net 131 "Net-(BZ1-Pad1)"))
+    (model ${KISYS3DMOD}/Diode_THT.3dshapes/D_DO-41_SOD81_P7.62mm_Horizontal.wrl
+      (at (xyz 0 0 0))
+      (scale (xyz 1 1 1))
+      (rotate (xyz 0 0 0))
+    )
+  )
   (module Connector_PinHeader_2.54mm:PinHeader_1x02_P2.54mm_Horizontal (layer F.Cu)
     (at 66 136 180)
@@
   (segment (start 110 141.0747) (end 112.5 143.5747) (width 0.25) (layer B.Cu) (net 92))
   (segment (start 97 89.7) (end 97 77) (width 0.25) (layer F.Cu) (net 130) (status 30))
+  (segment (start 97.456 89.244) (end 97 89.7) (width 0.25) (layer F.Cu) (net 130))
+  (segment (start 112.435 89.244) (end 97.456 89.244) (width 0.25) (layer F.Cu) (net 130))
   (segment (start 97 96.3) (end 82.84 96.3) (width 0.25) (layer F.Cu) (net 131) (status 30))
   (segment (start 82.84 96.3) (end 82.54 96) (width 0.25) (layer F.Cu) (net 131) (status 30))
+  (segment (start 97.564 96.864) (end 97 96.3) (width 0.25) (layer F.Cu) (net 131))
+  (segment (start 112.435 96.864) (end 97.564 96.864) (width 0.25) (layer F.Cu) (net 131))
   (segment (start 83.352 147.29) (end 80.812 147.29) (width 0.25) (layer F.Cu) (net 132) (status 30))
   (segment (start 85.892 147.29) (end 83.352 147.29) (width 0.25) (layer F.Cu) (net 132) (status 30))
